File: head-sensor-board.kicad_sch (KiCad schematic)
At the start: 0 parts

Commit message: Stage 2: schematic (ERC 0), custom libs, BOM, verification tools
- Schematic (KiCad 10, A3, 40 parts): XIAO ESP32S3 on 2x7 sockets, VL53L1X
  headers J1/J2 (jumper wires; pin order is a PLACEHOLDER, unverified),
  2 LED channels (NSSW157T + AO3400A, PWM) with external LED headers J3/J4,
  per-channel solder jumper SJ1/SJ2 selecting 3V3 (R1/R2 20 ohm 0603, default)
  or 5V (R3/R4 33 ohm 2010), pull-ups (XSHUT fitted, I2C DNP), 8 test points,
  decoupling, M2 holes. Design notes with the LED / 3V3 / GPIO calculations
  are in the schematic itself.
- ERC: 0 errors, 0 warnings; strict run (4 normally-ignored checks enabled): 0.
- tools/check_netlist.py: 25/25 nets match the intended netlist; every
  schematic pin exists as a pad in its footprint.
- libs/: XIAO_ESP32S3, ToF_Header_1x06, Q_NMOS_GSD symbols; XIAO THT 2x7 and
  NSSW157T footprints (sources in README).
- docs/spec.md rewritten for Stage 2 (user answers applied; 3V3 total incl.
  Wi-Fi/camera peaks; MOSFET gate drive check; 5V resistor selection),
  docs/bom.md + bom.csv, ERC reports, schematic PDF.

Co-Authored-By: Claude Sonnet 5.5 <noreply@anthropic.com>
Parts:
- added C1: 10u, Capacitor_SMD:C_0805_2012Metric, symbol Device:C
- added C2, C3: 100n, Capacitor_SMD:C_0603_1608Metric, symbol Device:C
- added D1, D2: NSSW157T, head-sensor-board:LED_Nichia_NSSW157T, symbol Device:LED
- added H1, H2: MountingHole_2.2mm_M2, MountingHole:MountingHole_2.2mm_M2, symbol Mechanical:MountingHole
- added J1: ToF_L (PLACEHOLDER), Connector_PinHeader_2.54mm:PinHeader_1x06_P2.54mm_Vertical, symbol head-sensor-board:ToF_Header_1x06
- added J2: ToF_R (PLACEHOLDER), Connector_PinHeader_2.54mm:PinHeader_1x06_P2.54mm_Vertical, symbol head-sensor-board:ToF_Header_1x06
- added J3: LED_L_EXT (1:+ 2:-), Connector_PinHeader_2.54mm:PinHeader_1x02_P2.54mm_Vertical, symbol Connector_Generic:Conn_01x02
- added J4: LED_R_EXT (1:+ 2:-), Connector_PinHeader_2.54mm:PinHeader_1x02_P2.54mm_Vertical, symbol Connector_Generic:Conn_01x02
- added Q1, Q2: AO3400A, Package_TO_SOT_SMD:SOT-23, symbol head-sensor-board:Q_NMOS_GSD
- added R1, R2: 20, Resistor_SMD:R_0603_1608Metric, symbol Device:R
- added R10, R9: 1, Resistor_SMD:R_0603_1608Metric, symbol Device:R
- added R11, R12: 10k, Resistor_SMD:R_0603_1608Metric, symbol Device:R
- added R13, R14: 3.3k, Resistor_SMD:R_0603_1608Metric, symbol Device:R
- added R15, R16: 0, Resistor_SMD:R_0603_1608Metric, symbol Device:R
- added R3, R4: 33, Resistor_SMD:R_2010_5025Metric, symbol Device:R
- added R5, R6: 220, Resistor_SMD:R_0603_1608Metric, symbol Device:R
- added R7, R8: 100k, Resistor_SMD:R_0603_1608Metric, symbol Device:R
- added SJ1: LED_L_SUPPLY, Jumper:SolderJumper-3_P1.3mm_Bridged12_RoundedPad1.0x1.5mm, symbol Jumper:SolderJumper_3_Bridged12
- added SJ2: LED_R_SUPPLY, Jumper:SolderJumper-3_P1.3mm_Bridged12_RoundedPad1.0x1.5mm, symbol Jumper:SolderJumper_3_Bridged12
- added TP1: 3V3, TestPoint:TestPoint_Pad_D1.5mm, symbol Connector:TestPoint
- added TP2: GND, TestPoint:TestPoint_Pad_D1.5mm, symbol Connector:TestPoint
- added TP3: SCL, TestPoint:TestPoint_Pad_D1.5mm, symbol Connector:TestPoint
- added TP4: SDA, TestPoint:TestPoint_Pad_D1.5mm, symbol Connector:TestPoint
- added TP5: XSHUT_L, TestPoint:TestPoint_Pad_D1.5mm, symbol Connector:TestPoint
- added TP6: XSHUT_R, TestPoint:TestPoint_Pad_D1.5mm, symbol Connector:TestPoint
- added TP7: ILED_L, TestPoint:TestPoint_Pad_D1.5mm, symbol Connector:TestPoint
- added TP8: ILED_R, TestPoint:TestPoint_Pad_D1.5mm, symbol Connector:TestPoint
- added U1: XIAO_ESP32S3_Sense, head-sensor-board:XIAO_ESP32S3_THT_2x7_P2.54mm, symbol head-sensor-board:XIAO_ESP32S3
Connections:
- new net: R3.2, SJ1.3 (B)
- new net: R2.2, SJ2.1 (A)
- new net: R1.2, SJ1.1 (A)
- new net: R4.2, SJ2.3 (B)
- new net +3V3: C1.1, C2.1, C3.1, J1.1 (VIN), J2.1 (VIN), R1.1, R11.1, R12.1, R13.1, R14.1, R2.1, TP1.1, U1.12 (3V3)
- new net +5V: R3.1, R4.1, U1.14 (5V)
- new net D8_GPIO7: R15.1, U1.9 (D8/SCK)
- new net D9_GPIO8: R16.1, U1.10 (D9/MISO)
- new net GATE_L: Q1.1 (G), R5.2, R7.1
- new net GATE_R: Q2.1 (G), R6.2, R8.1
- new net GND: C1.2, C2.2, C3.2, J1.2 (GND), J2.2 (GND), R10.2, R7.2, R8.2, R9.2, TP2.1, U1.13 (GND)
- new net LEDA_L: D1.2 (A), J3.1 (Pin_1), SJ1.2 (C)
- new net LEDA_R: D2.2 (A), J4.1 (Pin_1), SJ2.2 (C)
- new net LEDK_L: D1.1 (K), J3.2 (Pin_2), Q1.3 (D)
- new net LEDK_R: D2.1 (K), J4.2 (Pin_2), Q2.3 (D)
- new net LED_PWM_L: R5.1, U1.3 (D2)
- new net LED_PWM_R: R6.1, U1.4 (D3)
- new net SCL: J1.3 (SCL), J2.3 (SCL), R14.2, TP3.1, U1.6 (D5/SCL)
- new net SDA: J1.4 (SDA), J2.4 (SDA), R13.2, TP4.1, U1.5 (D4/SDA)
- new net SENSE_L: Q1.2 (S), R9.1, TP7.1
- new net SENSE_R: Q2.2 (S), R10.1, TP8.1
- new net TOF_L_INT: J1.6 (GPIO1), R15.2
- new net TOF_R_INT: J2.6 (GPIO1), R16.2
- new net XSHUT_L: J1.5 (XSHUT), R11.2, TP5.1, U1.1 (D0)
- new net XSHUT_R: J2.5 (XSHUT), R12.2, TP6.1, U1.2 (D1)
- no-connect marks 0 -> 3
Other:
- note added: "0.33 mA. ESP32-S3: IOH 40 mA / IOL 28 mA (Datasheet v2.2 Table 5-4)."
- note added: "0.65-1.45 V, Rds(on) < 48 mohm @2.5 V."
- note added: "3.3 V gate drive is enough: ESP32-S3 VOH >= 0.8*VDD = 2.64 V. AO3400A (AOS Rev 3.1): VGS(th)"
- note added: "3V3"
- note added: "5V"
- note added: "5V total with the XIAO webcam capture peak 347 mA (Seeed wiki) = 493 mA (< 500 mA USB 2.0). XIAO 5V pin current capability: UNVERIFIED."
- note added: "= 6 / 16 / 26 % of IF max 150 mA = 11 / 30 / 49 % of the 80 mA rated flux."
- note added: "=> Measure the real 5V input current before running Wi-Fi TX + capture + LEDs 100 % + ToF peak"
- note added: "A. POWER"
- note added: "B. LED @3V3 (R1/R2 20 ohm 0603)"
- note added: "Both SOT-23, pin 1=G 2=S 3=D."
- note added: "C. LED @5V (R3/R4 33 ohm 2010 0.5 W)"
- note added: "D. 3V3 TOTAL (Seeed: 'You can draw 700mA', condition not stated)"
- note added: "D0=GPIO1 XSHUT_L | D1=GPIO2 XSHUT_R | D2=GPIO3 LED_L PWM (strapping pin, gate pulled low) | D3=GPIO4 LED_R PWM"
- note added: "D4=GPIO5 SDA | D5=GPIO6 SCL | D6/D7=GPIO43/44 reserved UART | D8/D9=GPIO7/8 = ToF GPIO1 via DNP links R15/R16 (shared with Sense"
- note added: "D6/TX, D7/RX: reserved (UART to body XIAO)"
- note added: "Decoupling (3V3)"
- note added: "Do NOT short J3/J4 + to -: R1 would dissipate 0.49 W (0603 = 0.1 W), R3 0.71 W (2010 = 0.5 W)."
- note added: "E. GPIO and MOSFET gate drive"
- note added: "Everything is powered from the XIAO 3V3 pin. XIAO 5V pin is wired ONLY to R3/R4 -> solder jumper pad 3 (open by default)."
- note added: "External: LEDs 77.6 + ToF peak 2 x 40 + XSHUT pull-ups 0.7 = 158 mA (81 mA if the LEDs are on 5V)."
- note added: "F. GPIO assignment (approved 2026-10-01)"
- note added: "Fi TX peak 340 mA (chip only, Datasheet v2.2 Table 5-7)."
- note added: "Firmware: drive both XSHUT low first, release one at a time and change the VL53L1X address (default 0x29 7-bit = 0x52 8-bit)."
- note added: "For 5V: cut the 1-2 bridge, bridge 2-3 (R3/R4 33 ohm 2010 are already fitted). 5V = USB VBUS (no voltage on battery power)."
- note added: "G. UNVERIFIED / WARNINGS"
- note added: "GPIO carries no LED current (gate only). Gate charge peak 3.3 V / 220 ohm = 15 mA; XSHUT low sinks"
- note added: "Header pin order = PLACEHOLDER (UNVERIFIED)"
- note added: "J3/J4 external LED: pin 1 = + (after the series resistor), pin 2 = -. Fit EITHER D1/D2 or an external LED (both = they share the current)."
- note added: "LED channel L"
- note added: "LED channel R"
- note added: "LED supply per channel: SJ1/SJ2 default = pads 1-2 bridged = 3V3 via R1/R2 (20 ohm)."
- note added: "M2 mounting holes x2 (placed on the board in Stage 3)"
- note added: "MCU: XIAO ESP32S3 Sense (2x7 sockets or pin headers)"
- note added: "NOTES (full calculation: docs/spec.md, tools/led_budget.py)"
- note added: "Pull-ups"
- note added: "R1/R2 dissipation <= 30 mW (30 % of 0.1 W). Both LEDs at 100 % duty, max: 77.6 mA."
- note added: "R13/R14: DNP (I2C pull-ups)"
- note added: "Seeed camera table MAX ~0.65 A (conditions not stated = UNVERIFIED) -> 808 mA (115 %). ESP32-S3 Wi-"
- note added: "Si2302CDS (Vishay S12-2336 Rev D): VGS(th) 0.40-0.85 V, Rds(on) < 75 mohm @2.5 V, VGS max +-8 V."
- note added: "Test points"
- note added: "ToF header pin order is a PLACEHOLDER (module not in hand). Gerbers are NOT released until the real pinout is checked. ToF modules are wired with"
- note added: "ToF modules (jumper wires)"
- note added: "Vcc 3.2-3.4 V (assumed), Rds(on) <= 75 mohm. Per LED min/nom/max = 8.5 / 23.6 / 38.8 mA"
- note added: "Vcc 4.75-5.25 V: 45.0 / 59.0 / 73.0 mA per LED (49 % of IF max). R3/R4 dissipation <= 176 mW (35 % of 0.5 W)."
- note added: "Vf(I) = 2.677 V + 5.29 ohm*I (Nichia STS-DA1-1913: 3.1 V typ and 2.8-3.4 V @80 mA; 2.73 V @10 mA read from the graph = reference only)."
- note added: "With the wrong resistor (20 ohm on 5V) a LED would get 109 mA and R1 238 mW -> always keep SJ and R1/R3 as drawn."
- note added: "XIAO Sense (Seeed wiki): webcam average 140 mA, capture peak 366 mA -> total 524 mA (75 % of 700"
- note added: "jumper wires."
- note added: "mA)."
- note added: "microSD) | 5V: SJ option only"
- note added: "together."
- company: (none) -> Serpens / Floor Watch
- title: (none) -> head-sensor-board

Commit message: Stage 3: board outline 40x25 mm and component placement (no routing)
- tools/gen_pcb.py (KiCad bundled Python): builds the board from the schematic
  netlist: outline with variable W/H/corner R/hole inset, M2 holes, footprints
  with nets, symbol fields and schematic links, silkscreen labels, back legend.
  Edge usage: USB-C at the left edge, LEDs D1/D2 and external LED headers
  J3/J4 at the right/long edges, ToF headers J1/J2 on the top/bottom long
  edges, test points on the top face (ILED TPs + GND together).
  Small parts sit under the XIAO (courtyard limited to the pin-row strips).
- DRC with schematic parity: 0 errors / 0 warnings except 64 unconnected
  items (routing is Stage 4). 40x25 is the minimum for this arrangement
  (39.5 x 25 or 40 x 24.8 overlap).
- libs: XIAO courtyard = pin-row strips; new TestPoint_Pad_D1.5mm_NoSilk.
- schematic notes: add H (operating cautions: 5V is a test option, 493 mA is
  at the USB 2.0 limit; do not run Wi-Fi TX + capture + LEDs 100 % + ToF peak
  together until the real 5V input current is measured).
- docs: spec.md Stage 3 (placement, verification), README, placement images,
  drc_report.txt.

Co-Authored-By: Claude Sonnet 5.5 <noreply@anthropic.com>
Parts:
- TP1, TP2, TP3, TP4, TP5, TP6, TP7, TP8: footprint TestPoint:TestPoint_Pad_D1.5mm -> head-sensor-board:TestPoint_Pad_D1.5mm_NoSilk
Other:
- note added: "(margin 7 mA)."
- note added: "3V3: do NOT run Wi-Fi TX, camera capture, LEDs at 100 % and ToF peaks at"
- note added: "5V is a TEST OPTION only. The default is 3V3 (SJ1/SJ2 pads 1-2 bridged)."
- note added: "H. OPERATING CAUTIONS (user, 2026-10-01)"
- note added: "The 5V total of 493 mA is right at the USB 2.0 limit of 500 mA"
- note added: "measured."
- note added: "the same time, until the real 5V input current of the XIAO has been"
Changed lines of the file:
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@@
 			)
 		)
-		(property "Footprint" "TestPoint:TestPoint_Pad_D1.5mm"
+		(property "Footprint" "head-sensor-board:TestPoint_Pad_D1.5mm_NoSilk"
 			(at 299.72 97.79 0)
 			(hide yes)
@@
 			)
 		)
-		(property "Footprint" "TestPoint:TestPoint_Pad_D1.5mm"
+		(property "Footprint" "head-sensor-board:TestPoint_Pad_D1.5mm_NoSilk"
 			(at 382.27 97.79 0)
 			(hide yes)
@@
 			)
 		)
-		(property "Footprint" "TestPoint:TestPoint_Pad_D1.5mm"
+		(property "Footprint" "head-sensor-board:TestPoint_Pad_D1.5mm_NoSilk"
 			(at 46.99 162.56 0)
 			(hide yes)
@@
 			)
 		)
-		(property "Footprint" "TestPoint:TestPoint_Pad_D1.5mm"
+		(property "Footprint" "head-sensor-board:TestPoint_Pad_D1.5mm_NoSilk"
 			(at 62.23 162.56 0)
 			(hide yes)
@@
 			)
 		)
-		(property "Footprint" "TestPoint:TestPoint_Pad_D1.5mm"
+		(property "Footprint" "head-sensor-board:TestPoint_Pad_D1.5mm_NoSilk"
 			(at 77.47 162.56 0)
 			(hide yes)
@@
 			)
 		)
-		(property "Footprint" "TestPoint:TestPoint_Pad_D1.5mm"
+		(property "Footprint" "head-sensor-board:TestPoint_Pad_D1.5mm_NoSilk"
 			(at 92.71 162.56 0)
 			(hide yes)
@@
 			)
 		)
-		(property "Footprint" "TestPoint:TestPoint_Pad_D1.5mm"
+		(property "Footprint" "head-sensor-board:TestPoint_Pad_D1.5mm_NoSilk"
 			(at 107.95 162.56 0)
 			(hide yes)
@@
 			)
 		)
-		(property "Footprint" "TestPoint:TestPoint_Pad_D1.5mm"
+		(property "Footprint" "head-sensor-board:TestPoint_Pad_D1.5mm_NoSilk"
 			(at 123.19 162.56 0)
 			(hide yes)
@@
 		(effects
 			(font
+				(size 1.1 1.1)
+			)
+			(justify left bottom)
+		)
+	)
+	(text "H. OPERATING CAUTIONS (user, 2026-10-01)"
+		(exclude_from_sim no)
+		(at 207.86 255.9 0)
+		(effects
+			(font
+				(size 1.4 1.4)
+				(bold yes)
+			)
+			(justify left bottom)
+		)
+	)
+	(text "5V is a TEST OPTION only. The default is 3V3 (SJ1/SJ2 pads 1-2 bridged)."
+		(exclude_from_sim no)
+		(at 207.86 260.5 0)
+		(effects
+			(font
+				(size 1.1 1.1)
+			)
+			(justify left bottom)
+		)
+	)
+	(text "   The 5V total of 493 mA is right at the USB 2.0 limit of 500 mA"
+		(exclude_from_sim no)
+		(at 207.86 264.4 0)
+		(effects
+			(font
+				(size 1.1 1.1)
+			)
+			(justify left bottom)
+		)
+	)
+	(text "   (margin 7 mA)."
+		(exclude_from_sim no)
+		(at 207.86 268.3 0)
+		(effects
+			(font
+				(size 1.1 1.1)
+			)
+			(justify left bottom)
+		)
+	)
+	(text "3V3: do NOT run Wi-Fi TX, camera capture, LEDs at 100 % and ToF peaks at"
+		(exclude_from_sim no)
+		(at 207.86 272.2 0)
+		(effects
+			(font
+				(size 1.1 1.1)
+			)
+			(justify left bottom)
+		)
+	)
+	(text "   the same time, until the real 5V input current of the XIAO has been"
+		(exclude_from_sim no)
+		(at 207.86 276.1 0)
+		(effects
+			(font
+				(size 1.1 1.1)
+			)
+			(justify left bottom)
+		)
+	)
+	(text "   measured."
+		(exclude_from_sim no)
+		(at 207.86 280 0)
+		(effects
+			(font

Commit message: Stage 4: 44x28 mm board, routing, DRC 0, 3D views (no gerbers/BOM/pos yet)
- Board outline 44x28 mm (corner R1, M2 x2 unchanged); placement revised for routability
  (J1/J2 rotated so SDA/SCL match XIAO order, SJ vertical, R3/R4 split by channel, TP5/TP6 moved).
- Silkscreen: L / R, USB-C arrow, J1/J2 six signal names (VIN GND SCL SDA XSHUT GPIO1).
- Auto-router (tools/route.py: numpy+scipy grid Dijkstra) + apply_routes.py + make_board.py.
  Power 0.5 mm, LED current paths 0.4 mm, signals 0.25 mm, GND pour both sides, 30 vias.
- DRC (schematic parity, --severity-all): 0 violations, 0 unconnected, 0 mismatches.
  Previously-ignored checks (missing courtyard, type/filter mismatch, via centering) set to error.
- J1/J2 use project footprint PinHeader_1x06_P2.54mm_NoSilk (standard silk outline removed).
- Simple 3D models (3dmodels/, illustration only), KiCad 3D renders, routed placement PNG.
- README: ToF module pinout fields + jumper-wire correspondence table (to fill when the module arrives).
- Sense expansion board vs placed parts checked from Seeed drawings (spec 6.5); camera/microSD protrusion unverified.

Co-Authored-By: Claude Sonnet 5.5 <noreply@anthropic.com>
Parts:
- J1, J2: footprint Connector_PinHeader_2.54mm:PinHeader_1x06_P2.54mm_Vertical -> head-sensor-board:PinHeader_1x06_P2.54mm_NoSilk
Changed lines of the file:
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@@
 			)
 		)
-		(property "Footprint" "Connector_PinHeader_2.54mm:PinHeader_1x06_P2.54mm_Vertical"
+		(property "Footprint" "head-sensor-board:PinHeader_1x06_P2.54mm_NoSilk"
 			(at 200.66 66.04 0)
 			(hide yes)
@@
 			)
 		)
-		(property "Footprint" "Connector_PinHeader_2.54mm:PinHeader_1x06_P2.54mm_Vertical"
+		(property "Footprint" "head-sensor-board:PinHeader_1x06_P2.54mm_NoSilk"
 			(at 200.66 111.76 0)
 			(hide yes)
